Commit message: Add files via upload

File: race_it/description/inertial.xacro (robot description, xacro)
@@ -13,4 +13,5 @@
     <xacro:macro name="inertial_cylinder" params="mass length radius">
         <inertial>
+            <origin xyz="0 0 0" rpy="${-pi/2} 0 0"/>    <!--NEW-->
             <mass value="${mass}" />
             <inertia ixx="${(1/12) * mass * (3*radius*radius + length*length)}" ixy="0.0" ixz="0.0"

File: race_it/description/ros2_ack.xacro (robot description, xacro)
@@ -3,9 +3,11 @@
     <ros2_control name="carbot" type="system">
         <hardware>
-            <!-- <plugin>gazebo_ros2_control/GazeboSystem</plugin> -->
+            <plugin>gazebo_ros2_control/GazeboSystem</plugin>
+            <!--
             <plugin>ros2_control_demo_example_11/CarlikeBotSystemHardware</plugin>
             <param name="example_param_hw_start_duration_sec">0</param>
             <param name="example_param_hw_stop_duration_sec">3.0</param>
             <param name="is_simulation">1</param>
+            -->
         </hardware>
         <!-- Front Left Wheel -->
@@ -32,11 +34,10 @@
     <gazebo>
         <plugin filename="libgazebo_ros2_control.so" name="gazebo_ros2_control">
-            <!--
             <ros>
                 <remapping>asc/reference_unstamped:=cmd_vel</remapping>
                 <remapping>asc/odometry:=odom</remapping>
                 <remapping>asc/tf_odometry:=tf</remapping>
+                <robot_base_frame>base_link</robot_base_frame>
             </ros>
-            -->
             <parameters>$(find race_it)/config/controller/my_controllers.yaml</parameters>
         </plugin>

File: race_it/description/temp_controllers/carzzz.xacro (robot description, xacro)
@@ -4,11 +4,10 @@
 <!-- <xacro:include filename="gazebo_control_dd.xacro"/> -->
 <!-- <xacro:include filename="gazebo_control_steer.xacro"/> -->
-    <xacro:property name="wheel_width" value="0.026"/>
-    <xacro:property name="wheel_radius" value="0.033"/>
+    <xacro:property name="wheel_width" value="0.04"/>
+    <xacro:property name="wheel_radius" value="0.1"/>
     <!-- Wheel macro -->
     <xacro:macro name="wheel" params="name">
         <link name="${name}">
             <visual>
-                <origin xyz="0 0 0" rpy="${-pi/2} 0 0"/>    <!--NEW-->
                 <geometry>
                     <cylinder length="${wheel_width}" radius="${wheel_radius}" />
@@ -17,10 +16,9 @@
             </visual>
             <collision>
-                <origin xyz="0 0 0" rpy="${-pi/2} 0 0"/>    <!--NEW-->
                 <geometry>
                     <cylinder length="${wheel_width}" radius="${wheel_radius}" />
                 </geometry>
             </collision>
-            <xacro:inertial_cylinder mass="0.1" length="${wheel_width}" radius="${wheel_radius}"/>
+             <xacro:inertial_cylinder mass="0.1" length="${wheel_width}" radius="${wheel_radius}"/>
         </link>
         <gazebo reference="${name}">
@@ -28,11 +26,10 @@
         </gazebo>
     </xacro:macro>
-    <xacro:property name="hinge_width" value="0.008"/>
-    <xacro:property name="hinge_radius" value="0.0066"/>
+    <xacro:property name="hinge_width" value="0.04"/>
+    <xacro:property name="hinge_radius" value="0.02"/>
     <!-- Hinge macro -->
     <xacro:macro name="hinge" params="name">
         <link name="${name}">
             <visual>
-                <origin xyz="0 0 0" rpy="${-pi/2} 0 0"/>    <!--NEW-->
                 <geometry>
                     <cylinder length="${hinge_width}" radius="${hinge_radius}" />
@@ -41,10 +38,9 @@
             </visual>
             <collision>
-                <origin xyz="0 0 0" rpy="${-pi/2} 0 0"/>    <!--NEW-->
                 <geometry>
                     <cylinder length="${hinge_width}" radius="${hinge_radius}" />
                 </geometry>
             </collision>
-            <xacro:inertial_cylinder mass="0.1" length="${hinge_width}" radius="${hinge_radius}"/>
+             <xacro:inertial_cylinder mass="0.1" length="${hinge_width}" radius="${hinge_radius}"/>
         </link>
         <gazebo reference="${name}">
@@ -67,5 +63,5 @@
         <visual>
         <geometry>
-            <box size="0.4 0.2 0.1"/>
+            <box size="0.5 1.0 0.2"/>
         </geometry>
         <origin xyz="0 0 0" rpy="0 0 0"/>
@@ -74,8 +70,8 @@
         </material>
         </visual>
-        <xacro:inertial_box mass="0.5" x="0.4" y="0.2" z="0.1"/>
+        <xacro:inertial_box mass="0.5" x="0.5" y="1.0" z="0.15"/>
     </link>
     <gazebo reference="chassis_link">
-        <material>Gazebo/Orange</material>
+            <material>Gazebo/Orange</material>
     </gazebo>
     <!-- Base Chassis Joint -->
@@ -83,5 +79,5 @@
         <parent link="base_link"/>
         <child link="chassis_link"/>
-        <origin xyz="0 0 0.05" rpy="0 0 0 "/>
+        <origin xyz="0 0 0.2" rpy="0 0 0 "/>
     </joint>
     <!-- Front Left Hinge -->
@@ -91,7 +87,7 @@
             <child link="front_left_hinge"/>
             <!-- <origin xyz="-0.25 0.5 -0.1" rpy="0 ${-pi/2} 0"/> -->
-            <origin xyz="0.15 0.104 -0.05" rpy="0 0 0"/> <!--0.15 0.071 0.0-->
+            <origin xyz="-0.27 0.48 -0.08" rpy="0 ${-pi/2} 0"/>
             <limit upper="0.5236" lower="-0.5236" velocity="20" effort="1"/>
-            <axis xyz="0 0 1"/>
+            <axis xyz="1 0 0"/>
     </joint>
     <gazebo reference="front_left_hinge">
@@ -108,6 +104,6 @@
             <child link="front_left_link"/>
             <!-- <origin xyz="-0.25 0.5 -0.1" rpy="0 ${-pi/2} 0"/> -->
-            <origin xyz="0.0 0.017 0.0" rpy="0 0 0"/>
-            <axis xyz="0 1 0"/>
+            <origin xyz="0.0 0.0 0.04" rpy="0 0 0"/>
+            <axis xyz="0 0 1"/>
     </joint>
     <gazebo reference="front_left_link">
@@ -124,7 +120,7 @@
             <child link="front_right_hinge"/>
             <!-- <origin xyz="-0.25 0.5 -0.1" rpy="0 ${-pi/2} 0"/> -->
-            <origin xyz="0.15 -0.104 -0.05" rpy="0 0 0"/>  <!-- pi -->
+            <origin xyz="0.27 0.48 -0.08" rpy="0 ${-pi/2} 0"/>
             <limit upper="0.5236" lower="-0.5236" velocity="20" effort="1"/>
-            <axis xyz="0 0 1"/>
+            <axis xyz="1 0 0"/>
     </joint>
     <gazebo reference="front_right_hinge">
@@ -141,6 +137,6 @@
             <child link="front_right_link"/>
             <!-- <origin xyz="0.25 0.5 -0.1" rpy="0 ${-pi/2} 0"/> -->
-            <origin xyz="0.0 -0.017 0.0" rpy="0 0 0"/>
-            <axis xyz="0 1 0"/>
+            <origin xyz="0 0 -0.04" rpy="0 0 0"/>
+            <axis xyz="0 0 1"/>
     </joint>
     <gazebo reference="front_right_link">
@@ -156,6 +152,6 @@
             <parent link="chassis_link"/>
             <child link="rear_left_link"/>
-            <origin xyz = "-0.15 0.121 -0.05" rpy="0 0 0"/> <!--pi-->
-            <axis xyz="0 1 0"/>
+            <origin xyz="-0.31 -0.48 -0.08" rpy="0 ${-pi/2} 0"/>
+            <axis xyz="0 0 1"/>
     </joint>
     <!-- Rear Right Wheel -->
@@ -164,6 +160,6 @@
             <parent link="chassis_link"/>
             <child link="rear_right_link"/>
-            <origin xyz = "-0.15 -0.121 -0.05" rpy="0 0 0"/> <!-- pi    Default value for x is "0.27" -->
-            <axis xyz="0 1 0"/>
+            <origin xyz="0.31 -0.48 -0.08" rpy="0 ${-pi/2} 0"/> <!-- Default value for x is "0.27" -->
+            <axis xyz="0 0 1"/>
     </joint>
     <xacro:include filename="ros2_ack.xacro"/>
@@ -171,5 +167,5 @@
         <parent link="chassis_link"/>
         <child link="laser_frame"/>
-        <origin xyz="0.1 0.0 0.08" rpy="0 0 0"/>    <!--0 0.25 0.12-->
+        <origin xyz="0 0.25 0.12" rpy="0 0 0"/>    <!--0.1 0 0.175-->
     </joint>
     <link name="laser_frame">
@@ -185,5 +181,5 @@
             </geometry>
         </collision>
-        <xacro:Inertial_cylinder mass="0.0001" length="0.04" radius="0.05">
+        <xacro:Inertial_cylinder mass="0.1" length="0.04" radius="0.05">
             <origin xyz="0 0 0" rpy="0 0 0"/>
         </xacro:Inertial_cylinder>
